Commit message: Fixed sense of rotation of z axis in Tx200 ceiling mounted

File: bernina_urdf/tx200_ceiling.urdf (robot description, URDF)
Before this commit: robot staubli_tx200, 8 links, 7 joints
Joints:
- joint joint_1: axis 0 0 1 -> 0 0 -1
- joint joint_4: axis 0 0 1 -> 0 0 -1
- joint joint_6: axis 0 0 1 -> 0 0 -1

Commit message: added detector dummy to bernina robot

File: bernina_urdf/tx200_ceiling.urdf (robot description, URDF)
Before this commit: robot staubli_tx200, 8 links, 7 joints
Links:
- removed link tool0
- added link detector; visual box size=0.3 0.15 0.11
Joints:
- removed joint joint_6-tool0
- added joint joint_6-detetcor: type fixed, parent link_6, child detector, origin xyz=.25 0 2.15 rpy=0 3.141592653589793 0

Commit message: added 1.5M meshes

File: bernina_urdf/tx200_ceiling.urdf (robot description, URDF)
Before this commit: robot staubli_tx200, 8 links, 7 joints
Links:
- link detector: geometry visual mesh filename=meshes/staeubli_tx200/visual/detector_1.5M.dae
Joints:
- joint joint_6-detetcor: origin xyz=.25 0 2.15 rpy=0 3.141592653589793 0 -> xyz=.25 0 2.15 rpy=0 0. 0

Commit message: added linear axis and rail

File: bernina_urdf/tx200_ceiling.urdf (robot description, URDF)
Before this commit: robot staubli_tx200, 8 links, 7 joints
Links:
- added link adapter; visual mesh filename=meshes/staeubli_tx200/visual/tool_adapter_plate.dae
- added link linear_axis; visual mesh filename=meshes/staeubli_tx200/visual/linear_axis.dae
- added link rail; visual mesh filename=meshes/staeubli_tx200/visual/rail.dae
Joints:
- removed joint joint_6-detetcor
- added joint adapter-detetcor: type fixed, parent adapter, child detector, origin xyz=.0 0 0. rpy=0 0. 0
- added joint joint_6-adapter: type fixed, parent link_6, child adapter, origin xyz=0.25 0.0 2.15 rpy=0 0. 0
- added joint linear_axis-base_link: type fixed, parent linear_axis, child base_link, origin xyz=.0 0 0. rpy=0 0. 0
- added joint rail-linear: type prismatic, parent rail, child linear_axis, origin xyz=.0 0 0. rpy=0 0. 0, axis 1 0 0, limit lower=-2. upper=2. effort=692.0 velocity=2.

Commit message: minor changes

File: bernina_urdf/tx200_ceiling.urdf (robot description, URDF)
Before this commit: robot staubli_tx200, 11 links, 10 joints
Joints:
- joint linear_axis-base_link: origin xyz=.0 0 0. rpy=0 0. 0 -> xyz=.0 0 0. rpy=0 0. 3.141592653589793
- joint rail-linear: limit lower=-2. upper=2. effort=692.0 velocity=2. -> lower=-0.2 upper=4. effort=692.0 velocity=2.; origin xyz=.0 0 0. rpy=0 0. 0 -> xyz=-2.125 0 0. rpy=0 0. 0

Commit message: colored mesh of JF1.5M modules

File: bernina_urdf/tx200_ceiling.urdf (robot description, URDF)
Before this commit: robot staubli_tx200, 11 links, 10 joints
Links:
- added link modules; visual mesh filename=meshes/staeubli_tx200/visual/detector_1.5M_modules.dae
Joints:
- added joint detetcor-modules: type fixed, parent detector, child modules, origin xyz=.0 0 0. rpy=0 0. 0

Commit message: new smaller mesh models

File: bernina_urdf/tx200_ceiling.urdf (robot description, URDF)
Before this commit: robot staubli_tx200, 12 links, 11 joints
Links:
- link base_link: geometry visual mesh filename=meshes/staeubli_tx200/visual/base_link.stl
- link link_1: geometry visual mesh filename=meshes/staeubli_tx200/visual/link_1.stl
- link link_2: geometry visual mesh filename=meshes/staeubli_tx200/visual/link_2.stl
- link link_3: geometry visual mesh filename=meshes/staeubli_tx200/visual/link_3.stl
- link link_4: geometry visual mesh filename=meshes/staeubli_tx200/visual/link_4.stl
- link link_5: geometry visual mesh filename=meshes/staeubli_tx200/visual/link_5.stl
- link link_6: geometry visual mesh filename=meshes/staeubli_tx200/visual/link_6.stl

Commit message: changed mesh links

File: bernina_urdf/tx200_ceiling.urdf (robot description, URDF)
Before this commit: robot staubli_tx200, 12 links, 11 joints
Links:
- link base_link: geometry visual mesh filename=meshes/staeubli_tx200/visual/base_link_sm.dae
- link link_1: geometry visual mesh filename=meshes/staeubli_tx200/visual/link_1_sm.dae
- link link_2: geometry visual mesh filename=meshes/staeubli_tx200/visual/link_2_sm.dae
- link link_3: geometry visual mesh filename=meshes/staeubli_tx200/visual/link_3_sm.dae
- link link_4: geometry visual mesh filename=meshes/staeubli_tx200/visual/link_4_sm.dae
- link link_5: geometry visual mesh filename=meshes/staeubli_tx200/visual/link_5_sm.dae
- link link_6: geometry visual mesh filename=meshes/staeubli_tx200/visual/link_6_sm.dae

Commit message: added collision protection and 90deg rotated JF

File: bernina_urdf/tx200_ceiling.urdf (robot description, URDF)
Before this commit: robot staubli_tx200, 12 links, 11 joints
Links:
- link adapter: geometry visual mesh filename=meshes/staeubli_tx200/visual/tool_adapter_plate_col.dae
- link detector: geometry visual mesh filename=meshes/staeubli_tx200/visual/detector_1.5M_90.dae
- link modules: geometry visual mesh filename=meshes/staeubli_tx200/visual/detector_1.5M_modules_90.dae
