Commit message: corrected gps urdf file

File: bernina_urdf/gps_phi_stage_hex.urdf (robot description, URDF)
Before this commit: robot general purpose station, 9 links, 8 joints
Links:
- removed link thc
- added link bridge; visual mesh filename=meshes/gps/bridge.dae
- added link chamber; visual mesh filename=meshes/gps/chamber.dae
- link base: geometry visual mesh filename=meshes/gps/base.dae
- link eta_stage: geometry visual mesh filename=meshes/gps/transl_eta.dae
- link hexapod: geometry visual mesh filename=meshes/gps/hexapod.dae
- link platform: geometry visual mesh filename=meshes/gps/platform.dae
- link th_arm: geometry visual mesh filename=meshes/gps/theta_arm.dae
- link tth_arm: geometry visual mesh filename=meshes/gps/ttheta_arm.dae
Joints:
- removed joint rzbase
- removed joint thc
- added joint bridge: type fixed, parent tth_arm, child bridge, origin xyz=0 0 0. rpy=0 0. 0
- added joint rxbase: type revolute, parent ybase, child platform, origin xyz=0 0 0. rpy=0 0. 0, axis 0 1 0, limit lower=-1 upper=1. effort=692.0 velocity=2.
- added joint yhl: type fixed, parent bridge, child chamber, origin xyz=0 0 0. rpy=0 0. 0
- joint eta: axis 0 1 0 -> 0 -1 0; limit lower=-0.2 upper=4. effort=692.0 velocity=2. -> lower=-10. upper=10. effort=692.0 velocity=2.
- joint mu: limit lower=-0.2 upper=4. effort=692.0 velocity=2. -> lower=-3.14 upper=3.14 effort=692.0 velocity=2.
- joint nu: limit lower=-0.2 upper=4. effort=692.0 velocity=2. -> lower=-3.14 upper=3.14 effort=692.0 velocity=2.
- joint transl_eta: limit lower=-0.2 upper=4. effort=692.0 velocity=2. -> lower=-0.1 upper=4. effort=692.0 velocity=2.
- joint xbase: axis 1 0 0 -> 0 1 0

Commit message: corrected gps urdf file

File: bernina_urdf/gps_phi_stage_hex.urdf (robot description, URDF)
Before this commit: robot general purpose station, 10 links, 9 joints
Joints:
- joint eta: origin xyz=0 0 0. rpy=0 0. 0 -> xyz=0 0 0.68 rpy=0 0. 0

Commit message: committing changes to gps model

File: bernina_urdf/gps_phi_stage_hex.urdf (robot description, URDF)
Before this commit: robot general purpose station, 10 links, 9 joints
Links:
- removed link eta_stage
- removed link hexapod
- removed link platform
- removed link th_arm
- removed link tth_arm
- added link eta; visual mesh filename=meshes/gps/hexapod.dae
- added link gamma; visual mesh filename=meshes/gps/ttheta_arm.dae
- added link mu; visual mesh filename=meshes/gps/theta_arm.dae
- added link rxbase; visual mesh filename=meshes/gps/platform.dae
- added link transl_eta; visual mesh filename=meshes/gps/transl_eta.dae
Joints:
- removed joint nu
- added joint gamma: type revolute, parent rxbase, child gamma, origin xyz=0 0 0. rpy=0 0. 0, axis 0 0 1, limit lower=-3.14 upper=3.14 effort=692.0 velocity=2.
- joint bridge: parent tth_arm -> gamma
- joint eta: child hexapod -> eta; origin xyz=0 0 0.68 rpy=0 0. 0 -> xyz=0 0 1.42 rpy=0 0. 0; parent eta_stage -> transl_eta
- joint mu: child th_arm -> mu; parent platform -> rxbase
- joint rxbase: child platform -> rxbase
- joint transl_eta: child eta_stage -> transl_eta; parent th_arm -> mu

Commit message: corrected position of robot wrt origin

File: bernina_urdf/gps_phi_stage_hex.urdf (robot description, URDF)
Before this commit: robot general purpose station, 10 links, 9 joints
Joints:
- joint gamma: origin xyz=0 0 0. rpy=0 0. 0 -> xyz=0 0 0. rpy=0 0. -1.5707963

File: bernina_urdf/tx200_ceiling.urdf (robot description, URDF)
Before this commit: robot staubli_tx200, 12 links, 11 joints
Joints:
- joint rail-linear: origin xyz=-2.125 0 0. rpy=0 0. 0 -> xyz=-1.425 0. 0. rpy=0 0. 0

File: bernina_urdf/tx200_ceiling_16M.urdf (robot description, URDF)
Before this commit: robot staubli_tx200, 11 links, 10 joints
Joints:
- joint rail-linear: origin xyz=-2.125 0 0. rpy=0 0. 0 -> xyz=-1.425 0 0. rpy=0 0. 0
